File: pedal.kicad_pcb (KiCad board)
At the start: 2 copper layers, 50 x 60 mm, 50 parts, among them J1 Conn_01x01_Female, J2 Conn_01x01_Female, J3 Conn_01x02_Female, J4 Conn_01x02_Female, J5 Conn_01x01_Female, U1 L78L05_TO92, U2 NE5532D8R2G, U3 PT2399

Commit message: adding ground plane and other fixes
Parts:
- added G***: LOGO, lib:ninetales, B.Cu at (92.2, 99.8)
Connections:
- C4 pad 1: Earth -> Net-(R8-Pad1)
- C4 pad 2: Net-(C4-Pad2) -> Earth
- R8 pad 1: Net-(C4-Pad2) -> Net-(R8-Pad1)
- U1 pad 1: Net-(C4-Pad2) -> Net-(R8-Pad1)
- U3 pad 1: Net-(C4-Pad2) -> Net-(R8-Pad1)
Routing:
- net Net-(R8-Pad1): track 0.00 -> 50.1 mm
- net Net-(C4-Pad2): track 49.2 -> 0.00 mm
- net Earth: track 246.5 -> 253.1 mm
- net Net-(C6-Pad1): track 23.7 -> 24.6 mm
- net /outa: track 67.3 -> 66.7 mm
- added copper zone on B.Cu, net Earth
- added copper zone on F.Cu, net Earth
