File: pedal.kicad_sch (KiCad schematic)
At the start: 40 parts, among them U1 L78L05_TO92, U2 NE5532D8R2G, U3 PT2399

Commit message: doing the schematic
Parts:
- added H1, H2, H3, H4: MountingHole_Pad, MountingHole:MountingHole_3.2mm_M3_Pad_TopBottom, symbol Mechanical:MountingHole_Pad
- added J1, J2, J5: Conn_01x01_Female, Connector_PinHeader_2.54mm:PinHeader_1x01_P2.54mm_Vertical, symbol Connector:Conn_01x01_Female
- added J3, J4: Conn_01x02_Female, Connector_PinHeader_2.54mm:PinHeader_1x02_P2.54mm_Vertical, symbol Connector:Conn_01x02_Female
- added R21: 330, Resistor_THT:R_Axial_DIN0207_L6.3mm_D2.5mm_P10.16mm_Horizontal, symbol Device:R
- C1: footprint Capacitor_SMD:C_0603_1608Metric_Pad1.08x0.95mm_HandSolder -> Capacitor_THT:CP_Radial_D5.0mm_P2.50mm
- C10, C11, C12, C13, C14, C15, C2, C5, C7, C8, C9: footprint (none) -> Capacitor_THT:C_Disc_D4.3mm_W1.9mm_P5.00mm
- C3, C4, C6: footprint (none) -> Capacitor_THT:CP_Radial_D5.0mm_P2.50mm
- R1, R10, R11, R12, R13, R14, R15, R16, R17, R18, R19, R2, R3, R4, R5, R6, R7, R8, R9: footprint (none) -> Resistor_THT:R_Axial_DIN0207_L6.3mm_D2.5mm_P10.16mm_Horizontal
- R20: renamed from R?; footprint (none) -> Resistor_THT:R_Axial_DIN0207_L6.3mm_D2.5mm_P10.16mm_Horizontal
- RV1, RV2: footprint (none) -> TerminalBlock:TerminalBlock_bornier-3_P5.08mm
- U2: footprint SOIC-8_NB_ONS -> Package_DIP:DIP-8_W7.62mm_Socket_LongPads
- U3: footprint (none) -> Package_DIP:DIP-16_W7.62mm_Socket_LongPads
Connections:
- net Earth: now also H1.1, H2.1, H3.1, H4.1, J3.2 (Pin_2), J4.1 (Pin_1), J4.2 (Pin_2)
- net VCC: now also J3.1 (Pin_1), R21.1
- net at C5.1, R20.2: now also J1.1 (Pin_1)
- net at C14.2, C15.1, R19.2: now also J2.1 (Pin_1)
- new net: J5.1 (Pin_1), R21.2
Other:
- note added: "GND Pads"
- note added: "Input: 9V"
- note added: "LED Circuit"
- note added: "Mechanical"
- note added: "Power Input"
- moved on the sheet: C1, C10, C11, C12, C13, C14, C15, C2, C3, C4, C5, C6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

Commit message: minor fixes and project settings
Parts:
- R19: value 10k -> 100k
Connections:
- net Earth: now also C4.2; no longer C4.1
- net at R8.1, U1.1 (VO), U3.1 (VCC): now also C4.1; no longer C4.2
Other:
- company: (none) -> Author: Vitória Beatriz Bianchin
- title: (none) -> Little Angel Chorus 
- moved on the sheet: C4
Changed lines of the file:
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@@
 (kicad_sch (version 20211123) (generator eeschema)
   (paper "A4")
+  (title_block
+    (title "Little Angel Chorus ")
+    (date "2023-05-23")
+    (company "Author: Vitória Beatriz Bianchin")
+    (comment 1 "Email: vitoriabbianchin@gmail.com")
+    (comment 2 "Original schematic by Rick Holt ")
+  )
   (junction (at 139.7 97.79) (diameter 0) (color 0 0 0 0)
   )
@@
     (pin "2")
   )
-  (symbol (lib_id "Device:C_Polarized") (at 72.898 69.596 0) (unit 1)
-    (in_bom yes) (on_board yes) (fields_autoplaced)
-    (property "Reference" "C4" (id 0) (at 75.946 67.4369 0)
-      (effects (font (size 1.27 1.27)) (justify left))
-    )
-    (property "Value" "47uF" (id 1) (at 75.946 69.9769 0)
-      (effects (font (size 1.27 1.27)) (justify left))
-    )
-    (property "Footprint" "Capacitor_THT:CP_Radial_D5.0mm_P2.50mm" (id 2) (at 73.8632 73.406 0)
+  (symbol (lib_id "Device:C_Polarized") (at 72.898 69.596 180) (unit 1)
+    (in_bom yes) (on_board yes) (fields_autoplaced)
+    (property "Reference" "C4" (id 0) (at 76.2 69.2149 0)
+      (effects (font (size 1.27 1.27)) (justify right))
+    )
+    (property "Value" "47uF" (id 1) (at 76.2 71.7549 0)
+      (effects (font (size 1.27 1.27)) (justify right))
+    )
+    (property "Footprint" "Capacitor_THT:CP_Radial_D5.0mm_P2.50mm" (id 2) (at 71.9328 65.786 0)
       (effects (font (size 1.27 1.27)) hide)
     )
@@
     (in_bom yes) (on_board yes)
     (property "Reference" "R19" (id 0) (at 173.99 60.6736 0))
-    (property "Value" "10k" (id 1) (at 173.99 58.6416 0))
+    (property "Value" "100k" (id 1) (at 173.99 58.6416 0))
     (property "Footprint" "Resistor_THT:R_Axial_DIN0207_L6.3mm_D2.5mm_P10.16mm_Horizontal" (id 2) (at 179.07 59.6576 90)
       (effects (font (size 1.27 1.27)) hide)
@@
     )
     (path "/d71891e5-c312-4665-a42b-045b28fe68e5"
-      (reference "R19") (unit 1) (value "10k") (footprint "Resistor_THT:R_Axial_DIN0207_L6.3mm_D2.5mm_P10.16mm_Horizontal")
+      (reference "R19") (unit 1) (value "100k") (footprint "Resistor_THT:R_Axial_DIN0207_L6.3mm_D2.5mm_P10.16mm_Horizontal")
     )
     (path "/6a98e60f-af7b-4c1a-9441-3d8b95a7c539"
